Commit message: add mecanum wheel suppurt in gazebo

File: modules/rover0/src/rover0_description/ros2_control/rover0.ros2_control.xacro (robot description, xacro)
@@ -7,5 +7,7 @@
             <plugin>gz_ros2_control/GazeboSimSystem</plugin>
         </xacro:if>
-        <plugin>rover0_hardware_interface/Rover0HardwareInterface</plugin>
+        <xacro:if value="false">
+            <plugin>rover0_hardware_interface/Rover0HardwareInterface</plugin>
+        </xacro:if>
         <param name="front_left_wheel_joint_name">front_left_wheel_joint</param>
         <param name="front_right_wheel_joint_name">front_right_wheel_joint</param>

File: modules/rover0/src/rover0_description/urdf/rover0_description.urdf.xacro (robot description, xacro)
@@ -1,4 +1,4 @@
 <?xml version="1.0"?>
-<robot xmlns:xacro="http://www.ros.org/wiki/xacro">
+<robot xmlns:xacro="http://www.ros.org/wiki/xacro" xmlns:gz="http://gazebosim.org/schema">
   <xacro:macro name="rover0" params="prefix">
     <xacro:property name="PI" value="3.1415926535897931"/>
@@ -20,5 +20,5 @@
     <xacro:macro name="box_inertia" params="m w h d">
       <inertial>
-        <origin xyz="0 0 0" rpy="${pi/2} 0 ${pi/2}"/>
+        <origin xyz="0 0 0" rpy="0 0 0"/>
         <mass value="${m}"/>
         <inertia ixx="${(m/12) * (h*h + d*d)}" ixy="0.0" ixz="0.0" iyy="${(m/12) * (w*w + d*d)}" iyz="0.0" izz="${(m/12) * (w*w + h*h)}"/>
@@ -27,5 +27,5 @@
     <xacro:macro name="cylinder_inertia" params="m r h">
       <inertial>
-        <origin xyz="0 0 0" rpy="${pi/2} 0 0" />
+        <origin xyz="0 0 0" rpy="0 0 0" />
         <mass value="${m}"/>
         <inertia ixx="${(m/12) * (3*r*r + h*h)}" ixy = "0" ixz = "0" iyy="${(m/12) * (3*r*r + h*h)}" iyz = "0" izz="${(m/2) * (r*r)}"/>
@@ -79,11 +79,11 @@
         <xacro:cylinder_inertia m="0.5" r="${wheel_radius}" h="${wheel_width}"/>
         <collision>
-          <origin xyz="0 0 0" rpy="${pi/2} 0 0"/>
+          <origin xyz="0 0 0" rpy="0 0 0"/>
           <geometry>
-            <cylinder radius="${wheel_radius}" length="${wheel_width}"/>
+            <sphere radius="${wheel_radius}"/>
           </geometry>
         </collision>
         <visual>
-          <origin xyz="0 0 0" rpy="${pi/2} 0 0"/>
+          <origin xyz="0 0 0" rpy="0 0 0"/>
           <geometry>
             <cylinder radius="${wheel_radius}" length="${wheel_width}"/>
@@ -95,7 +95,20 @@
         <parent link="base_link" />
         <child link="${prefix}_link" />
-        <origin xyz="${x_reflect*wheel_xoff} ${y_reflect * (base_width/2 + wheel_ygap)} ${-wheel_zoff}" rpy="0 0 0" />
-        <axis xyz="0 1 0" />
+        <origin xyz="${x_reflect*wheel_xoff} ${y_reflect * (base_width/2 + wheel_ygap)} ${-wheel_zoff}" rpy="-${pi/2} 0 0" />
+        <axis xyz="0 0 1" />
       </joint>
+      <gazebo reference="${prefix}_link">
+        <collision>
+          <surface>
+            <friction>
+              <ode>
+                <mu>1.0</mu>
+                <mu2>0.0</mu2>
+                <fdir1 gz:expressed_in="base_footprint"> 1 ${-x_reflect*y_reflect} 0</fdir1>
+              </ode>
+            </friction>
+          </surface>
+        </collision>
+      </gazebo>
     </xacro:macro>
     <xacro:wheel prefix="front_left_wheel" x_reflect="1" y_reflect="1" />
@@ -258,13 +271,4 @@
     </gazebo>
     <gazebo>
-        <plugin
-            filename="gz-sim-velocity-control-system"
-            name="gz::sim::systems::VelocityControl">
-            <topic>mecanum_drive_controller/cmd_vel</topic>
-            <initial_linear>0 0 0</initial_linear>
-            <initial_angular>0 0 0</initial_angular>
-        </plugin>
-    </gazebo>
-    <gazebo>
         <plugin filename="gz_ros2_control-system" name="gz_ros2_control::GazeboSimROS2ControlPlugin">
             <parameters>$(find rover0_bringup)/config/rover0_controllers.yaml</parameters>

Commit message: simplify xacro files

File: modules/rover0/src/rover0_description/ros2_control/rover0.ros2_control.xacro (robot description, xacro)
@@ -4,10 +4,5 @@
     <ros2_control name="${name}" type="system">
       <hardware>
-        <xacro:if value="true">
-            <plugin>gz_ros2_control/GazeboSimSystem</plugin>
-        </xacro:if>
-        <xacro:if value="false">
-            <plugin>rover0_hardware_interface/Rover0HardwareInterface</plugin>
-        </xacro:if>
+        <xacro:insert_block name="hardware_system"/>
         <param name="front_left_wheel_joint_name">front_left_wheel_joint</param>
         <param name="front_right_wheel_joint_name">front_right_wheel_joint</param>
@@ -15,12 +10,4 @@
         <param name="rear_right_wheel_joint_name">rear_right_wheel_joint</param>
         <param name="imu_sensor_name">imu_sensor</param>
-        <param name="serial_port">/dev/ttyUSB0</param>
-        <param name="encoder_tics_per_revolution">64</param>
-        <param name="imu_linear_acceleration_offset_x">-0.04001879692077637</param>
-        <param name="imu_linear_acceleration_offset_y">-0.011276155710220337</param>
-        <param name="imu_linear_acceleration_offset_z">0.9002845287322998</param>
-        <param name="imu_angular_velocity_offset_x">-6.8362923339009285</param>
-        <param name="imu_angular_velocity_offset_y">0.2556564286351204</param>
-        <param name="imu_angular_velocity_offset_z">0.06320327520370483</param>
       </hardware>
       <joint name="${prefix}front_left_wheel_joint">

File: modules/rover0/src/rover0_description/urdf/rover0.urdf.xacro (robot description, xacro)
@@ -8,5 +8,23 @@
   <!-- Import Rover0 ros2_control description -->
   <xacro:include filename="$(find rover0_description)/ros2_control/rover0.ros2_control.xacro" />
-  <xacro:rover0 prefix="$(arg prefix)" />
-  <xacro:rover0_ros2_control name="Rover0" prefix="$(arg prefix)"/>
+  <!-- xacro:rover0 prefix="$(arg prefix)" /-->
+  <xacro:call macro="rover0" prefix="$(arg prefix)" />
+  <xacro:rover0_ros2_control name="Rover0" prefix="$(arg prefix)">
+    <xacro:property name="hardware_system">
+      <xacro:if value="false">
+          <plugin>gz_ros2_control/GazeboSimSystem</plugin>
+      </xacro:if>
+      <xacro:if value="true">
+          <plugin>rover0_hardware_interface/Rover0HardwareInterface</plugin>
+          <param name="serial_port">/dev/ttyUSB0</param>
+          <param name="encoder_tics_per_revolution">64</param>
+          <param name="imu_linear_acceleration_offset_x">-0.04001879692077637</param>
+          <param name="imu_linear_acceleration_offset_y">-0.011276155710220337</param>
+          <param name="imu_linear_acceleration_offset_z">0.9002845287322998</param>
+          <param name="imu_angular_velocity_offset_x">-6.8362923339009285</param>
+          <param name="imu_angular_velocity_offset_y">0.2556564286351204</param>
+          <param name="imu_angular_velocity_offset_z">0.06320327520370483</param>
+      </xacro:if>
+    </xacro:property>
+  </xacro:rover0_ros2_control>
 </robot>

File: modules/rover0/src/rover0_description/urdf/rover0_description.urdf.xacro (robot description, xacro)
@@ -2,4 +2,9 @@
 <robot xmlns:xacro="http://www.ros.org/wiki/xacro" xmlns:gz="http://gazebosim.org/schema">
   <xacro:macro name="rover0" params="prefix">
+    <xacro:include filename="$(find rover0_description)/urdf/rover0_description_common.urdf.xacro" />
+    <xacro:include filename="$(find rover0_description)/urdf/rover0_description_lidar.urdf.xacro" />
+    <xacro:include filename="$(find rover0_description)/urdf/rover0_description_imu.urdf.xacro" />
+    <xacro:include filename="$(find rover0_description)/urdf/rover0_description_camera.urdf.xacro" />
+    <xacro:include filename="$(find rover0_description)/urdf/rover0_description_wheel.urdf.xacro" />
     <xacro:property name="PI" value="3.1415926535897931"/>
     <xacro:property name="base_width" value="0.14" />
@@ -7,162 +12,65 @@
     <xacro:property name="base_height" value="0.058" />
     <xacro:property name="base_mass" value="0.3" />
-    <xacro:property name="wheel_radius" value="0.028" />
-    <xacro:property name="wheel_width" value="0.025" />
     <xacro:property name="wheel_ygap" value="0.01" />
-    <xacro:property name="wheel_zoff" value="0.021" />
-    <xacro:property name="wheel_xoff" value="0.055" />
-    <xacro:property name="wheel_mass" value="0.3" />
-    <xacro:property name="lidar_mount_height" value="0.092" />
-    <xacro:property name="lidar_mount_xoff" value="-0.078" />
-    <xacro:property name="lidar_height" value="0.032" />
-    <xacro:property name="lidar_radius" value="0.034" />
-    <!-- Define inertial property macros  -->
-    <xacro:macro name="box_inertia" params="m w h d">
-      <inertial>
-        <origin xyz="0 0 0" rpy="0 0 0"/>
-        <mass value="${m}"/>
-        <inertia ixx="${(m/12) * (h*h + d*d)}" ixy="0.0" ixz="0.0" iyy="${(m/12) * (w*w + d*d)}" iyz="0.0" izz="${(m/12) * (w*w + h*h)}"/>
-      </inertial>
+    <xacro:property name="wheel_x_off" value="0.055" />
+    <xacro:property name="wheel_y_off" value="${base_width/2 + wheel_ygap}" />
+    <xacro:property name="wheel_z_off" value="0.021" />
+    <xacro:property name="lidar_x_off" value="-0.078" />
+    <xacro:property name="camera_x_off" value="0.11" />
+    <xacro:property name="camera_y_off" value="0.0" />
+    <xacro:property name="camera_z_off" value="0.015" />
+    <xacro:macro name="base">
+        <link name="${prefix}base_link">
+          <visual>
+            <geometry>
+              <box size="${base_length} ${base_width} ${base_height}"/>
+            </geometry>
+            <material name="orange"/>
+          </visual>
+          <collision>
+            <geometry>
+              <box size="${base_length} ${base_width} ${base_height}"/>
+            </geometry>
+          </collision>
+          <xacro:box_inertia m="15" w="${base_width}" d="${base_length}" h="${base_height}"/>
+        </link>
+        <link name="${prefix}base_footprint" />
+        <joint name="${prefix}base_joint" type="fixed">
+          <parent link="base_footprint" />
+          <child link="base_link" />
+          <origin xyz="0.0 0.0 ${(wheel_radius+wheel_z_off)}" rpy="0 0 0" />
+        </joint>
     </xacro:macro>
-    <xacro:macro name="cylinder_inertia" params="m r h">
-      <inertial>
-        <origin xyz="0 0 0" rpy="0 0 0" />
-        <mass value="${m}"/>
-        <inertia ixx="${(m/12) * (3*r*r + h*h)}" ixy = "0" ixz = "0" iyy="${(m/12) * (3*r*r + h*h)}" iyz = "0" izz="${(m/2) * (r*r)}"/>
-      </inertial>
-    </xacro:macro>
-    <xacro:macro name="sphere_inertia" params="m r">
-      <inertial>
-        <mass value="${m}"/>
-        <inertia ixx="${(2/5) * m * (r*r)}" ixy="0.0" ixz="0.0" iyy="${(2/5) * m * (r*r)}" iyz="0.0" izz="${(2/5) * m * (r*r)}"/>
-      </inertial>
-    </xacro:macro>
-    <gazebo>
-        <plugin filename="gz-sim-joint-state-publisher-system"
-        name="gz::sim::systems::JointStatePublisher">
-          <topic>joint_states</topic>
-          <update>20</update>
-          <gz_frame_id>base_link</gz_frame_id>
-          <frame_id>base_link</frame_id>
-          <joint_name>front_left_wheel_joint</joint_name>
-          <joint_name>front_right_wheel_joint</joint_name>
-          <joint_name>rear_left_wheel_joint</joint_name>
-          <joint_name>rear_right_wheel_joint</joint_name>
-        </plugin>
-    </gazebo>
-    <!-- Base Link -->
-    <link name="${prefix}base_link">
-      <visual>
-        <geometry>
-          <box size="${base_length} ${base_width} ${base_height}"/>
-        </geometry>
-        <material name="orange"/>
-      </visual>
-      <collision>
-        <geometry>
-          <box size="${base_length} ${base_width} ${base_height}"/>
-        </geometry>
-      </collision>
-      <xacro:box_inertia m="15" w="${base_width}" d="${base_length}" h="${base_height}"/>
-    </link>
-    <link name="${prefix}base_footprint" />
+    <xacro:base/>
+    <xacro:wheel prefix="front_left" parent="base_link" x_reflect="1" y_reflect="1" x_off="${wheel_x_off}" y_off="${wheel_y_off}" z_off="${wheel_z_off}"/>
+    <xacro:wheel prefix="front_right" parent="base_link"  x_reflect="1" y_reflect="-1" x_off="${wheel_x_off}" y_off="${wheel_y_off}" z_off="${wheel_z_off}"/>
+    <xacro:wheel prefix="rear_left" parent="base_link" x_reflect="-1" y_reflect="1" x_off="${wheel_x_off}" y_off="${wheel_y_off}" z_off="${wheel_z_off}"/>
+    <xacro:wheel prefix="rear_right" parent="base_link" x_reflect="-1" y_reflect="-1" x_off="${wheel_x_off}" y_off="${wheel_y_off}" z_off="${wheel_z_off}"/>
+    <xacro:lidar prefix="rover0" parent="base_link" x_off="${lidar_x_off}" />
+    <xacro:imu prefix="rover0" parent="base_link" x_off="0" y_off="0" z_off="0"/>
+    <xacro:camera prefix="rover0" parent="base_link" x_off="${camera_x_off}" y_off="${camera_y_off}" z_off="${camera_z_off}"/>
     <gazebo reference="${prefix}base_footprint">
         <turnGravityOff>false</turnGravityOff>
     </gazebo>
-    <joint name="${prefix}base_joint" type="fixed">
-      <parent link="base_footprint" />
-      <child link="base_link" />
-      <origin xyz="0.0 0.0 ${(wheel_radius+wheel_zoff)}" rpy="0 0 0" />
-    </joint>
-    <xacro:macro name="wheel" params="prefix x_reflect y_reflect">
-      <link name="${prefix}_link">
-        <xacro:cylinder_inertia m="0.5" r="${wheel_radius}" h="${wheel_width}"/>
-        <collision>
-          <origin xyz="0 0 0" rpy="0 0 0"/>
-          <geometry>
-            <sphere radius="${wheel_radius}"/>
-          </geometry>
-        </collision>
-        <visual>
-          <origin xyz="0 0 0" rpy="0 0 0"/>
-          <geometry>
-            <cylinder radius="${wheel_radius}" length="${wheel_width}"/>
-          </geometry>
-          <material name="black" />
-        </visual>
-      </link>
-      <joint name="${prefix}_joint" type="continuous">
-        <parent link="base_link" />
-        <child link="${prefix}_link" />
-        <origin xyz="${x_reflect*wheel_xoff} ${y_reflect * (base_width/2 + wheel_ygap)} ${-wheel_zoff}" rpy="-${pi/2} 0 0" />
-        <axis xyz="0 0 1" />
-      </joint>
-      <gazebo reference="${prefix}_link">
-        <collision>
-          <surface>
-            <friction>
-              <ode>
-                <mu>1.0</mu>
-                <mu2>0.0</mu2>
-                <fdir1 gz:expressed_in="base_footprint"> 1 ${-x_reflect*y_reflect} 0</fdir1>
-              </ode>
-            </friction>
-          </surface>
-        </collision>
-      </gazebo>
+    <xacro:macro name="gz_wheel" params="prefix x_reflect y_reflect">
+        <gazebo reference="${prefix}_link">
+          <collision>
+            <surface>
+              <friction>
+                <ode>
+                  <mu>1.0</mu>
+                  <mu2>0.0</mu2>
+                  <fdir1 gz:expressed_in="base_footprint"> 1 ${-x_reflect*y_reflect} 0</fdir1>
+                </ode>
+              </friction>
+            </surface>
+          </collision>
+        </gazebo>
     </xacro:macro>
-    <xacro:wheel prefix="front_left_wheel" x_reflect="1" y_reflect="1" />
-    <xacro:wheel prefix="front_right_wheel" x_reflect="1" y_reflect="-1" />
-    <xacro:wheel prefix="rear_left_wheel" x_reflect="-1" y_reflect="1" />
-    <xacro:wheel prefix="rear_right_wheel" x_reflect="-1" y_reflect="-1" />
-    <link name="lidar_mount_link">
-      <inertial>
-        <origin xyz="0 0 0" rpy="0 0 0"/>
-        <mass value="0.125"/>
-        <inertia ixx="0.001"  ixy="0"  ixz="0" iyy="0.001" iyz="0" izz="0.001" />
-      </inertial>
-      <collision>
-        <origin xyz="0 0 0" rpy="0 0 0"/>
-        <geometry>
-            <box size="0.02 0.02 ${lidar_mount_height}"/>
-        </geometry>
-      </collision>
-      <visual>
-        <origin xyz="0 0 0" rpy="0 0 0"/>
-        <geometry>
-            <box size="0.02 0.02 ${lidar_mount_height}"/>
-        </geometry>
-      </visual>
-    </link>
-    <joint name="lidar_mount_joint" type="fixed">
-        <parent link="base_link"/>
-        <child link="lidar_mount_link"/>
-        <origin xyz="${lidar_mount_xoff} 0 ${(base_height + lidar_mount_height)/2}" rpy="0 0 0"/>
-    </joint>
-    <link name="lidar_link">
-      <inertial>
-        <origin xyz="0 0 0" rpy="0 0 0"/>
-        <mass value="0.125"/>
-        <inertia ixx="0.001"  ixy="0"  ixz="0" iyy="0.001" iyz="0" izz="0.001" />
-      </inertial>
-      <collision>
-        <origin xyz="0 0 0" rpy="0 0 0"/>
-        <geometry>
-            <cylinder radius="${lidar_radius}" length="${lidar_height}"/>
-        </geometry>
-      </collision>
-      <visual>
-        <origin xyz="0 0 0" rpy="0 0 0"/>
-        <geometry>
-            <cylinder radius="${lidar_radius}" length="${lidar_height}"/>
-        </geometry>
-      </visual>
-    </link>
-    <joint name="lidar_joint" type="fixed">
-        <parent link="lidar_mount_link"/>
-        <child link="lidar_link"/>
-        <origin xyz="0 0 ${(lidar_mount_height + lidar_height) / 2}" rpy="0 0 0"/>
-    </joint>
-    <gazebo reference="lidar_link">
+    <xacro:gz_wheel prefix="front_left_wheel" x_reflect="1" y_reflect="1" />
+    <xacro:gz_wheel prefix="front_right_wheel" x_reflect="1" y_reflect="-1" />
+    <xacro:gz_wheel prefix="rear_left_wheel" x_reflect="-1" y_reflect="1" />
+    <xacro:gz_wheel prefix="rear_right_wheel" x_reflect="-1" y_reflect="-1" />
+    <!-- gazebo reference="lidar_link">
         <sensor name="lidar" type="gpu_lidar">
             <always_on>true</always_on>
@@ -193,26 +101,6 @@
             </lidar>
         </sensor>
-    </gazebo>
-    <link name="imu_link">
-      <xacro:box_inertia m="0.01" w="0.01" d="0.01" h="0.001" />
-      <collision>
-        <origin xyz="0 0 0" rpy="0 0 0"/>
-        <geometry>
-          <box size="0.01 0.01 0.001"/>
-        </geometry>
-      </collision>
-      <visual>
-        <origin xyz="0 0 0" rpy="0 0 0"/>
-        <geometry>
-          <box size="0.01 0.01 0.001"/>
-        </geometry>
-      </visual>
-    </link>
-    <joint name="imu_joint" type="fixed">
-      <parent link="base_link"/>
-      <child link="imu_link"/>
-      <origin xyz="0 0 0.0"/> <!-- TODO: update correct value -->
-    </joint>
-    <gazebo reference="imu_link">
+    </gazebo -->
+    <!-- gazebo reference="imu_link">
       <sensor name="imu_sensor" type="imu">
         <always_on>true</always_on>
@@ -222,25 +110,5 @@
         <topic>imu</topic>
       </sensor>
-    </gazebo>
-    <link name="camera_link">
-      <xacro:box_inertia m="0.01" w="0.01" d="0.01" h="0.001" />
-      <collision>
-        <origin xyz="0 0 0" rpy="0 0 0"/>
-        <geometry>
-          <box size="0.01 0.01 0.001"/>
-        </geometry>
-      </collision>
-      <visual>
-        <origin xyz="0 0 0" rpy="0 0 0"/>
-        <geometry>
-          <box size="0.01 0.01 0.001"/>
-        </geometry>
-      </visual>
-    </link>
-    <joint name="camera_joint" type="fixed">
-      <parent link="base_link"/>
-      <child link="camera_link"/>
-      <origin xyz="0.11 0 0.015"/>
-    </joint>
+    </gazebo -->
     <gazebo reference="camera_link">
       <sensor name="camera" type="camera">
@@ -277,4 +145,15 @@
             </ros>
         </plugin>
+        <plugin filename="gz-sim-joint-state-publisher-system"
+        name="gz::sim::systems::JointStatePublisher">
+          <topic>joint_states</topic>
+          <update>20</update>
+          <gz_frame_id>base_link</gz_frame_id>
+          <frame_id>base_link</frame_id>
+          <joint_name>front_left_wheel_joint</joint_name>
+          <joint_name>front_right_wheel_joint</joint_name>
+          <joint_name>rear_left_wheel_joint</joint_name>
+          <joint_name>rear_right_wheel_joint</joint_name>
+        </plugin>
     </gazebo>
   </xacro:macro>
