Commit message: split rover0_description
The one is for real robot. And the other is for gazebo

File: modules/rover0/src/rover0_description/urdf/rover0.urdf.xacro (robot description, xacro)
@@ -2,29 +2,6 @@
 <robot xmlns:xacro="http://www.ros.org/wiki/xacro" name="rover0">
   <xacro:arg name="prefix" default="" />
-  <!-- Import Rover0 macro -->
+  <xacro:include filename="$(find rover0_description)/urdf/rover0.materials.xacro" />
   <xacro:include filename="$(find rover0_description)/urdf/rover0_description.urdf.xacro" />
-  <!-- Import Rviz colors -->
-  <xacro:include filename="$(find rover0_description)/urdf/rover0.materials.xacro" />
-  <!-- Import Rover0 ros2_control description -->
-  <xacro:include filename="$(find rover0_description)/ros2_control/rover0.ros2_control.xacro" />
-  <!-- xacro:rover0 prefix="$(arg prefix)" /-->
   <xacro:call macro="rover0" prefix="$(arg prefix)" />
-  <xacro:rover0_ros2_control name="Rover0" prefix="$(arg prefix)">
-    <xacro:property name="hardware_system">
-      <xacro:if value="false">
-          <plugin>gz_ros2_control/GazeboSimSystem</plugin>
-      </xacro:if>
-      <xacro:if value="true">
-          <plugin>rover0_hardware_interface/Rover0HardwareInterface</plugin>
-          <param name="serial_port">/dev/ttyUSB0</param>
-          <param name="encoder_tics_per_revolution">64</param>
-          <param name="imu_linear_acceleration_offset_x">-0.04001879692077637</param>
-          <param name="imu_linear_acceleration_offset_y">-0.011276155710220337</param>
-          <param name="imu_linear_acceleration_offset_z">0.9002845287322998</param>
-          <param name="imu_angular_velocity_offset_x">-6.8362923339009285</param>
-          <param name="imu_angular_velocity_offset_y">0.2556564286351204</param>
-          <param name="imu_angular_velocity_offset_z">0.06320327520370483</param>
-      </xacro:if>
-    </xacro:property>
-  </xacro:rover0_ros2_control>
 </robot>

File: modules/rover0/src/rover0_description/urdf/rover0_description.urdf.xacro (robot description, xacro)
@@ -1,23 +1,22 @@
 <?xml version="1.0"?>
-<robot xmlns:xacro="http://www.ros.org/wiki/xacro" xmlns:gz="http://gazebosim.org/schema">
+<robot xmlns:xacro="http://www.ros.org/wiki/xacro">
+   <xacro:include filename="$(find rover0_description)/urdf/rover0_description_common.urdf.xacro" />
+   <xacro:include filename="$(find rover0_description)/urdf/rover0_description_lidar.urdf.xacro" />
+   <xacro:include filename="$(find rover0_description)/urdf/rover0_description_imu.urdf.xacro" />
+   <xacro:include filename="$(find rover0_description)/urdf/rover0_description_camera.urdf.xacro" />
+   <xacro:include filename="$(find rover0_description)/urdf/rover0_description_wheel.urdf.xacro" />
+   <xacro:property name="base_width" value="0.14" />
+   <xacro:property name="base_length" value="0.255" />
+   <xacro:property name="base_height" value="0.058" />
+   <xacro:property name="base_mass" value="0.3" />
+   <xacro:property name="wheel_ygap" value="0.01" />
+   <xacro:property name="wheel_x_off" value="0.055" />
+   <xacro:property name="wheel_y_off" value="${base_width/2 + wheel_ygap}" />
+   <xacro:property name="wheel_z_off" value="0.021" />
+   <xacro:property name="lidar_x_off" value="-0.078" />
+   <xacro:property name="camera_x_off" value="0.11" />
+   <xacro:property name="camera_y_off" value="0.0" />
+   <xacro:property name="camera_z_off" value="0.015" />
   <xacro:macro name="rover0" params="prefix">
-    <xacro:include filename="$(find rover0_description)/urdf/rover0_description_common.urdf.xacro" />
-    <xacro:include filename="$(find rover0_description)/urdf/rover0_description_lidar.urdf.xacro" />
-    <xacro:include filename="$(find rover0_description)/urdf/rover0_description_imu.urdf.xacro" />
-    <xacro:include filename="$(find rover0_description)/urdf/rover0_description_camera.urdf.xacro" />
-    <xacro:include filename="$(find rover0_description)/urdf/rover0_description_wheel.urdf.xacro" />
-    <xacro:property name="PI" value="3.1415926535897931"/>
-    <xacro:property name="base_width" value="0.14" />
-    <xacro:property name="base_length" value="0.255" />
-    <xacro:property name="base_height" value="0.058" />
-    <xacro:property name="base_mass" value="0.3" />
-    <xacro:property name="wheel_ygap" value="0.01" />
-    <xacro:property name="wheel_x_off" value="0.055" />
-    <xacro:property name="wheel_y_off" value="${base_width/2 + wheel_ygap}" />
-    <xacro:property name="wheel_z_off" value="0.021" />
-    <xacro:property name="lidar_x_off" value="-0.078" />
-    <xacro:property name="camera_x_off" value="0.11" />
-    <xacro:property name="camera_y_off" value="0.0" />
-    <xacro:property name="camera_z_off" value="0.015" />
     <xacro:macro name="base">
         <link name="${prefix}base_link">
@@ -37,124 +36,17 @@
         <link name="${prefix}base_footprint" />
         <joint name="${prefix}base_joint" type="fixed">
-          <parent link="base_footprint" />
-          <child link="base_link" />
+          <parent link="${prefix}base_footprint" />
+          <child link="${prefix}base_link" />
           <origin xyz="0.0 0.0 ${(wheel_radius+wheel_z_off)}" rpy="0 0 0" />
         </joint>
     </xacro:macro>
     <xacro:base/>
-    <xacro:wheel prefix="front_left" parent="base_link" x_reflect="1" y_reflect="1" x_off="${wheel_x_off}" y_off="${wheel_y_off}" z_off="${wheel_z_off}"/>
-    <xacro:wheel prefix="front_right" parent="base_link"  x_reflect="1" y_reflect="-1" x_off="${wheel_x_off}" y_off="${wheel_y_off}" z_off="${wheel_z_off}"/>
-    <xacro:wheel prefix="rear_left" parent="base_link" x_reflect="-1" y_reflect="1" x_off="${wheel_x_off}" y_off="${wheel_y_off}" z_off="${wheel_z_off}"/>
-    <xacro:wheel prefix="rear_right" parent="base_link" x_reflect="-1" y_reflect="-1" x_off="${wheel_x_off}" y_off="${wheel_y_off}" z_off="${wheel_z_off}"/>
-    <xacro:lidar prefix="rover0" parent="base_link" x_off="${lidar_x_off}" />
-    <xacro:imu prefix="rover0" parent="base_link" x_off="0" y_off="0" z_off="0"/>
-    <xacro:camera prefix="rover0" parent="base_link" x_off="${camera_x_off}" y_off="${camera_y_off}" z_off="${camera_z_off}"/>
-    <gazebo reference="${prefix}base_footprint">
-        <turnGravityOff>false</turnGravityOff>
-    </gazebo>
-    <xacro:macro name="gz_wheel" params="prefix x_reflect y_reflect">
-        <gazebo reference="${prefix}_link">
-          <collision>
-            <surface>
-              <friction>
-                <ode>
-                  <mu>1.0</mu>
-                  <mu2>0.0</mu2>
-                  <fdir1 gz:expressed_in="base_footprint"> 1 ${-x_reflect*y_reflect} 0</fdir1>
-                </ode>
-              </friction>
-            </surface>
-          </collision>
-        </gazebo>
-    </xacro:macro>
-    <xacro:gz_wheel prefix="front_left_wheel" x_reflect="1" y_reflect="1" />
-    <xacro:gz_wheel prefix="front_right_wheel" x_reflect="1" y_reflect="-1" />
-    <xacro:gz_wheel prefix="rear_left_wheel" x_reflect="-1" y_reflect="1" />
-    <xacro:gz_wheel prefix="rear_right_wheel" x_reflect="-1" y_reflect="-1" />
-    <!-- gazebo reference="lidar_link">
-        <sensor name="lidar" type="gpu_lidar">
-            <always_on>true</always_on>
-            <visualize>true</visualize>
-            <update_rate>1</update_rate>
-            <topic>scan</topic>
-            <gz_frame_id>lidar_link</gz_frame_id>
-            <pose>${lidar_mount_xoff} 0 ${lidar_mount_height + (base_height + lidar_height) / 2} 0 0 0</pose>
-            <lidar>
-                <scan>
-                    <horizontal>
-                        <samples>360</samples>
-                        <resolution>1.0</resolution>
-                        <min_angle>0.00</min_angle>
-                        <max_angle>6.28</max_angle>
-                    </horizontal>
-                </scan>
-                <range>
-                    <min>0.12</min>
-                    <max>5.0</max>
-                    <resolution>0.015</resolution>
-                </range>
-                <noise>
-                    <type>gaussian</type>
-                    <mean>0.0</mean>
-                    <stddev>0.01</stddev>
-                </noise>
-            </lidar>
-        </sensor>
-    </gazebo -->
-    <!-- gazebo reference="imu_link">
-      <sensor name="imu_sensor" type="imu">
-        <always_on>true</always_on>
-        <visualize>true</visualize>
-        <update_rate>100</update_rate>
-        <gz_frame_id>imu_link</gz_frame_id>
-        <topic>imu</topic>
-      </sensor>
-    </gazebo -->
-    <gazebo reference="camera_link">
-      <sensor name="camera" type="camera">
-        <always_on>true</always_on>
-        <visualize>true</visualize>
-        <update_rate>30</update_rate>
-        <gz_frame_id>camera_link</gz_frame_id>
-        <topic>camera</topic>
-        <camera name="rpcam">
-          <camera_info_topic>camera/camera_info</camera_info_topic>
-          <horizontal_fov>1.089</horizontal_fov>
-          <image>
-              <width>640</width>
-              <height>480</height>
-              <format>R8G8B8</format>
-          </image>
-          <clip>
-              <near>0.1</near>
-              <far>100</far>
-          </clip>
-          <noise>
-              <type>gaussian</type>
-              <mean>0.0</mean>
-              <stddev>0.007</stddev>
-          </noise>
-        </camera>
-      </sensor>
-    </gazebo>
-    <gazebo>
-        <plugin filename="gz_ros2_control-system" name="gz_ros2_control::GazeboSimROS2ControlPlugin">
-            <parameters>$(find rover0_bringup)/config/rover0_controllers.yaml</parameters>
-            <ros>
-                <remapping>/controller_manager/robot_description:=/robot_description</remapping>
-            </ros>
-        </plugin>
-        <plugin filename="gz-sim-joint-state-publisher-system"
-        name="gz::sim::systems::JointStatePublisher">
-          <topic>joint_states</topic>
-          <update>20</update>
-          <gz_frame_id>base_link</gz_frame_id>
-          <frame_id>base_link</frame_id>
-          <joint_name>front_left_wheel_joint</joint_name>
-          <joint_name>front_right_wheel_joint</joint_name>
-          <joint_name>rear_left_wheel_joint</joint_name>
-          <joint_name>rear_right_wheel_joint</joint_name>
-        </plugin>
-    </gazebo>
+    <xacro:wheel prefix="front_left" parent="${prefix}base_link" x_reflect="1" y_reflect="1" x_off="${wheel_x_off}" y_off="${wheel_y_off}" z_off="${wheel_z_off}"/>
+    <xacro:wheel prefix="front_right" parent="${prefix}base_link"  x_reflect="1" y_reflect="-1" x_off="${wheel_x_off}" y_off="${wheel_y_off}" z_off="${wheel_z_off}"/>
+    <xacro:wheel prefix="rear_left" parent="${prefix}base_link" x_reflect="-1" y_reflect="1" x_off="${wheel_x_off}" y_off="${wheel_y_off}" z_off="${wheel_z_off}"/>
+    <xacro:wheel prefix="rear_right" parent="${prefix}base_link" x_reflect="-1" y_reflect="-1" x_off="${wheel_x_off}" y_off="${wheel_y_off}" z_off="${wheel_z_off}"/>
+    <xacro:lidar prefix="rover0" parent="${prefix}base_link" base_height="${base_height}" x_off="${lidar_x_off}" />
+    <xacro:imu prefix="rover0" parent="${prefix}base_link" x_off="0" y_off="0" z_off="0"/>
+    <xacro:camera prefix="rover0" parent="${prefix}base_link" x_off="${camera_x_off}" y_off="${camera_y_off}" z_off="${camera_z_off}"/>
   </xacro:macro>
 </robot>

File: modules/rover0/src/rover0_description/urdf/rover0_description_common.urdf.xacro (robot description, xacro)
@@ -1,4 +1,5 @@
 <?xml version="1.0"?>
-<robot xmlns:xacro="http://www.ros.org/wiki/xacro" xmlns:gz="http://gazebosim.org/schema">
+<robot xmlns:xacro="http://www.ros.org/wiki/xacro">
+    <xacro:property name="PI" value="3.1415926535897931"/>
     <xacro:macro name="box_inertia" params="m w h d">
       <inertial>

File: modules/rover0/src/rover0_description/urdf/rover0_description_imu.urdf.xacro (robot description, xacro)
@@ -1,4 +1,4 @@
 <?xml version="1.0"?>
-<robot xmlns:xacro="http://www.ros.org/wiki/xacro" xmlns:gz="http://gazebosim.org/schema">
+<robot xmlns:xacro="http://www.ros.org/wiki/xacro">
     <xacro:include filename="$(find rover0_description)/urdf/rover0_description_common.urdf.xacro" />
     <xacro:macro name="imu" params="prefix parent x_off y_off z_off">

File: modules/rover0/src/rover0_description/urdf/rover0_description_lidar.urdf.xacro (robot description, xacro)
@@ -1,9 +1,9 @@
 <?xml version="1.0"?>
-<robot xmlns:xacro="http://www.ros.org/wiki/xacro" xmlns:gz="http://gazebosim.org/schema">
+<robot xmlns:xacro="http://www.ros.org/wiki/xacro">
     <xacro:include filename="$(find rover0_description)/urdf/rover0_description_common.urdf.xacro" />
     <xacro:property name="mount_height" value="0.092" />
     <xacro:property name="lidar_height" value="0.032" />
     <xacro:property name="lidar_radius" value="0.034" />
-    <xacro:macro name="lidar" params="prefix parent x_off">
+    <xacro:macro name="lidar" params="prefix parent base_height x_off">
         <link name="${prefix}_lidar_mount_link">
           <inertial>

File: modules/rover0/src/rover0_description/urdf/rover0_description_wheel.urdf.xacro (robot description, xacro)
@@ -1,8 +1,9 @@
 <?xml version="1.0"?>
-<robot xmlns:xacro="http://www.ros.org/wiki/xacro" xmlns:gz="http://gazebosim.org/schema">
+<robot xmlns:xacro="http://www.ros.org/wiki/xacro">
     <xacro:include filename="$(find rover0_description)/urdf/rover0_description_common.urdf.xacro" />
     <xacro:property name="wheel_mass" value="0.3" />
     <xacro:property name="wheel_radius" value="0.028" />
     <xacro:property name="wheel_width" value="0.025" />
+    <xacro:property name="PI" value="3.1415926535897931"/>
     <xacro:macro name="wheel" params="prefix parent x_reflect y_reflect x_off y_off z_off">
       <link name="${prefix}_wheel_link">
