Commit message: improve ekf accuracy

File: modules/rover0/src/rover0_description/urdf/rover0_description_imu.urdf.xacro (robot description, xacro)
@@ -21,5 +21,6 @@
           <parent link="${parent}"/>
           <child link="${prefix}_imu_link"/>
-          <origin xyz="${x_off} ${y_off} ${z_off}"/> <!-- TODO: update correct value -->
+          <origin xyz="${x_off} ${y_off} ${z_off}" rpy="0 0 0"/> <!-- TODO: update correct value -->
+          <axis xyz="0 0 1"/>
         </joint>
     </xacro:macro>
