Commit message: fix lidar orientation

File: modules/rover0/src/rover0_description/urdf/rover0_description_lidar.urdf.xacro (robot description, xacro)
@@ -47,5 +47,5 @@
             <parent link="${parent}"/>
             <child link="${prefix}_lidar_mount_link"/>
-            <origin xyz="${x_off} 0 ${(base_height + mount_height)/2}" rpy="0 0 0"/>
+            <origin xyz="${x_off} 0 ${(base_height + mount_height)/2}" rpy="0 0 ${radians(180)}"/>
         </joint>
         <joint name="${prefix}_lidar_joint" type="fixed">

Commit message: fix lidar orientation

File: modules/rover0/src/rover0_description/urdf/rover0_description_lidar.urdf.xacro (robot description, xacro)
@@ -52,5 +52,5 @@
             <parent link="${prefix}_lidar_mount_link"/>
             <child link="${prefix}_lidar_link"/>
-            <origin xyz="0 0 ${(mount_height + lidar_height) / 2}" rpy="0 0 0"/>
+            <origin xyz="0 0 ${(mount_height + lidar_height) / 2}" rpy="0 ${radians(180)} 0"/>
         </joint>
     </xacro:macro>
